File: MCU_Datalogger.kicad_sch (KiCad schematic)
At the start: 25 parts, among them U1 24LC1025, U2 24LC1025, U3 DS1337S+T&R, U4 ATMEGA328P-AU, Y1 Crystal, Y2 Crystal

Commit message: valeurs des composants
Parts:
- C1, C3: value C -> 0.1uF
- C2, C4: value C -> 22pF
- C5: value Capacitor_PO -> 100nF
- R1, R2: value R -> 330
- R3, R6: value R -> 10K
- R4, R5: value R -> 4.7K
- Y1: value Crystal -> 32.768 KHz
- Y2: value Crystal -> 16 MHz
- renumbered R7 to 10K
Other:
- moved on the sheet: 10K, BT1, C1, C2, C3, C4, C5, D1, D2, H1, H2, H3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

Commit message: footprints
Parts:
- BT1: footprint (none) -> Connector_PinHeader_2.54mm:PinHeader_1x02_P2.54mm_Vertical
- C1, C2, C3, C4: footprint (none) -> Capacitor_SMD:C_0805_2012Metric
- C5: footprint Capacitor_THT:CP_Radial_D5.0mm_P2.50mm -> Capacitor_SMD:C_0805_2012Metric
- D1, D2: footprint LED_THT:LED_D5.0mm -> LED_SMD:LED_0805_2012Metric
- H1, H2, H3, H4: footprint (none) -> MountingHole:MountingHole_2.1mm
- R1, R2, R3, R4, R5, R6: footprint (none) -> Resistor_SMD:R_0805_2012Metric
- R7: renamed from 10K; value R -> 10K; footprint (none) -> Resistor_SMD:R_0805_2012Metric
- U1, U2: footprint (none) -> Package_SO:SOIC-8_5.23x5.23mm_P1.27mm
- U3: footprint SOIC127P600X175-8N -> footprints:SOIC127P600X175-8N
- U4: footprint QFP80P900X900X120-32N -> footprints:QFP80P900X900X120-32N
- Y1, Y2: footprint (none) -> Crystal:Crystal_SMD_5032-2Pin_5.0x3.2mm_HandSoldering
Changed lines of the file:
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@@
 			)
 		)
-		(property "Footprint" ""
+		(property "Footprint" "MountingHole:MountingHole_2.1mm"
 			(at 241.3 147.574 0)
 			(effects
@@
 			)
 		)
-		(property "Footprint" "LED_THT:LED_D5.0mm"
+		(property "Footprint" "LED_SMD:LED_0805_2012Metric"
 			(at 179.832 36.83 0)
 			(effects
@@
 			)
 		)
-		(property "Footprint" ""
+		(property "Footprint" "Resistor_SMD:R_0805_2012Metric"
 			(at 86.614 34.036 0)
 			(effects
@@
 			)
 		)
-		(property "Footprint" ""
+		(property "Footprint" "Resistor_SMD:R_0805_2012Metric"
 			(at 155.702 39.624 0)
 			(effects
@@
 			)
 		)
-		(property "Footprint" ""
+		(property "Footprint" "Resistor_SMD:R_0805_2012Metric"
 			(at 121.666 162.306 0)
 			(effects
@@
 			)
 		)
-		(property "Footprint" ""
+		(property "Footprint" "Package_SO:SOIC-8_5.23x5.23mm_P1.27mm"
 			(at 94.996 129.032 0)
 			(effects
@@
 			)
 		)
-		(property "Footprint" ""
+		(property "Footprint" "Capacitor_SMD:C_0805_2012Metric"
 			(at 175.768 22.606 0)
 			(effects
@@
 		(dnp no)
 		(fields_autoplaced yes)
-		(property "Reference" "10K"
+		(property "Reference" "R7"
 			(at 104.394 32.7659 0)
 			(effects
@@
 			)
 		)
-		(property "Value" "R"
+		(property "Value" "10K"
 			(at 104.394 35.3059 0)
 			(effects
@@
 			)
 		)
-		(property "Footprint" ""
+		(property "Footprint" "Resistor_SMD:R_0805_2012Metric"
 			(at 101.6 34.036 0)
 			(effects
@@
 			(project "MCU_Datalogger"
 				(path "/d9a5c4ae-f738-4eec-ba07-3147cf00a375"
-					(reference "10K")
+					(reference "R7")
 					(unit 1)
 				)
@@
 			)
 		)
-		(property "Footprint" ""
+		(property "Footprint" "Resistor_SMD:R_0805_2012Metric"
 			(at 137.922 162.56 0)
 			(effects
@@
 			)
 		)
-		(property "Footprint" ""
+		(property "Footprint" "Crystal:Crystal_SMD_5032-2Pin_5.0x3.2mm_HandSoldering"
 			(at 20.32 45.72 0)
 			(effects
@@
 			)
 		)
-		(property "Footprint" ""
+		(property "Footprint" "Resistor_SMD:R_0805_2012Metric"
 			(at 259.842 82.042 0)
 			(effects
@@
 			)
 		)
-		(property "Footprint" "Capacitor_THT:CP_Radial_D5.0mm_P2.50mm"
+		(property "Footprint" "Capacitor_SMD:C_0805_2012Metric"
 			(at 260.858 34.29 0)
 			(effects
@@
 			)
 		)
-		(property "Footprint" "QFP80P900X900X120-32N"
+		(property "Footprint" "footprints:QFP80P900X900X120-32N"
 			(at 215.646 56.388 0)
 			(effects
@@
 			)
 		)
-		(property "Footprint" ""
+		(property "Footprint" "Capacitor_SMD:C_0805_2012Metric"
 			(at 154.94 68.834 0)
 			(effects
@@
 			)
 		)
-		(property "Footprint" "LED_THT:LED_D5.0mm"
+		(property "Footprint" "LED_SMD:LED_0805_2012Metric"
 			(at 258.318 59.69 0)
 			(effects
@@
 			)
 		)
-		(property "Footprint" ""
+		(property "Footprint" "Package_SO:SOIC-8_5.23x5.23mm_P1.27mm"
 			(at 135.382 128.27 0)
 			(effects
@@
 			)
 		)
-		(property "Footprint" ""
+		(property "Footprint" "MountingHole:MountingHole_2.1mm"
 			(at 241.046 137.16 0)
 			(effects
@@
 			)
 		)
-		(property "Footprint" ""
+		(property "Footprint" "Resistor_SMD:R_0805_2012Metric"
 			(at 181.61 81.28 0)
 			(effects
@@
 			)
 		)
-		(property "Footprint" ""
+		(property "Footprint" "Capacitor_SMD:C_0805_2012Metric"
 			(at 115.316 35.814 0)
 			(effects
@@
 			)
 		)
-		(property "Footprint" ""
+		(property "Footprint" "MountingHole:MountingHole_2.1mm"
 			(at 240.792 127 0)
 			(effects
@@
 			)
 		)
-		(property "Footprint" ""
+		(property "Footprint" "Capacitor_SMD:C_0805_2012Metric"
 			(at 154.94 51.054 0)
 			(effects
@@
 			)
 		)
-		(property "Footprint" "SOIC127P600X175-8N"
+		(property "Footprint" "footprints:SOIC127P600X175-8N"
 			(at 52.832 44.704 0)
 			(effects
@@
 			)
 		)
-		(property "Footprint" ""
+		(property "Footprint" "Crystal:Crystal_SMD_5032-2Pin_5.0x3.2mm_HandSoldering"
 			(at 169.164 56.642 0)
 			(effects
@@
 			)
 		)
-		(property "Footprint" ""
+		(property "Footprint" "MountingHole:MountingHole_2.1mm"
 			(at 241.046 158.75 0)
 			(effects
@@
 			)
 		)
-		(property "Footprint" ""
+		(property "Footprint" "Connector_PinHeader_2.54mm:PinHeader_1x02_P2.54mm_Vertical"
 			(at 268.224 26.416 90)
 			(effects
